Commit message: Collision Ok

File: src/src/mlp3240/mlp3240_description/urdf/mlp3240_macro.xacro (robot description, xacro)
@@ -11,5 +11,5 @@
 			<mass value="0.01"/>
 			<inertia ixx="0.001" ixy="0.0" ixz="0.0" iyy="0.001" iyz="0.0" izz="0.001"/>
-		 </inertial>
+		</inertial>
 		<visual>
 		    <origin xyz="0 0 0" rpy="0 0 1.57" />
@@ -21,16 +21,17 @@
 		    </material>
 		</visual>
-	        <collision>
-		  <geometry>
-		    <mesh filename="package://mlp3240_description/mesh/visual/bottom.stl" scale="0.001 0.001 0.001"/>
-		  </geometry>
-	        </collision>
+	    <collision>
+		  	<origin xyz="0 0 0" rpy="0 0 1.57" />
+		  	<geometry>
+		    	<mesh filename="package://mlp3240_description/mesh/visual/bottom.stl" scale="0.001 0.001 0.001"/>
+		  	</geometry>
+	    </collision>
 	    </link>
 	    <link name="${prefix}left">
 	    	<inertial>
-			<origin xyz="0 0 0" rpy="0 0 0"/>
-			<mass value="0.001"/>
-			<inertia ixx="0.001" ixy="0.0" ixz="0.0" iyy="0.001" iyz="0.0" izz="0.001"/>
-		 </inertial>
+				<origin xyz="0 0 0" rpy="0 0 0"/>
+				<mass value="0.001"/>
+				<inertia ixx="0.001" ixy="0.0" ixz="0.0" iyy="0.001" iyz="0.0" izz="0.001"/>
+			</inertial>
 		<visual>
 		    <origin xyz="-0.01 0 0.014" rpy="0 0 1.57" />
@@ -42,16 +43,17 @@
 		    </material>
 		</visual>
-	        <collision>
-		  <geometry>
-		    <mesh filename="package://mlp3240_description/mesh/visual/lateral.stl" scale="0.001 0.001 0.001"/>
-		  </geometry>
-	        </collision>
+	    <collision>
+		  	<origin xyz="-0.01 0 0.014" rpy="0 0 1.57" />
+		  	<geometry>
+		    	<mesh filename="package://mlp3240_description/mesh/visual/lateral.stl" scale="0.001 0.001 0.001"/>
+		  	</geometry>
+	    </collision>
 	    </link>
 	    <link name="${prefix}right">
 	    	<inertial>
-			<origin xyz="0 0 0" rpy="0 0 0"/>
-			<mass value="0.001"/>
-			<inertia ixx="0.001" ixy="0.0" ixz="0.0" iyy="0.001" iyz="0.0" izz="0.001"/>
-		 </inertial>
+				<origin xyz="0 0 0" rpy="0 0 0"/>
+				<mass value="0.001"/>
+				<inertia ixx="0.001" ixy="0.0" ixz="0.0" iyy="0.001" iyz="0.0" izz="0.001"/>
+			</inertial>
 		<visual>
 		    <origin xyz="0.01 0 0.014" rpy="0 0 1.57" />
@@ -63,16 +65,17 @@
 		    </material>
 		</visual>
-	        <collision>
-		  <geometry>
-		    <mesh filename="package://mlp3240_description/mesh/visual/lateral.stl" scale="0.001 0.001 0.001"/>
-		  </geometry>
-	        </collision>
+	    <collision>
+			<origin xyz="0.01 0 0.014" rpy="0 0 1.57" />
+		    <geometry>
+		    	<mesh filename="package://mlp3240_description/mesh/visual/lateral.stl" scale="0.001 0.001 0.001"/>
+		  	</geometry>
+	    </collision>
 	    </link>
 	    <link name="${prefix}back">
 	    	<inertial>
-			<origin xyz="0 0 0" rpy="0 0 0"/>
-			<mass value="0.001"/>
-			<inertia ixx="0.001" ixy="0.0" ixz="0.0" iyy="0.001" iyz="0.0" izz="0.001"/>
-		 </inertial>
+				<origin xyz="0 0 0" rpy="0 0 0"/>
+				<mass value="0.001"/>
+				<inertia ixx="0.001" ixy="0.0" ixz="0.0" iyy="0.001" iyz="0.0" izz="0.001"/>
+			</inertial>
 		<visual>
 		    <origin xyz="0 -0.005 0.0065" rpy="0 0 1.57" />
@@ -85,15 +88,16 @@
 		</visual>
 		<collision>
-		  <geometry>
-		    <mesh filename="package://mlp3240_description/mesh/visual/front.stl" scale="0.001 0.001 0.001"/>
-		  </geometry>
-	        </collision>
+			<origin xyz="0 -0.005 0.0065" rpy="0 0 1.57" />
+		  	<geometry>
+		    	<mesh filename="package://mlp3240_description/mesh/visual/front.stl" scale="0.001 0.001 0.001"/>
+		 	</geometry>
+	    </collision>
 	    </link>
 	    <link name="${prefix}front">
 	    	<inertial>
-			<origin xyz="0 0 0" rpy="0 0 0"/>
-			<mass value="0.001"/>
-			<inertia ixx="0.001" ixy="0.0" ixz="0.0" iyy="0.001" iyz="0.0" izz="0.001"/>
-		 </inertial>
+				<origin xyz="0 0 0" rpy="0 0 0"/>
+				<mass value="0.001"/>
+				<inertia ixx="0.001" ixy="0.0" ixz="0.0" iyy="0.001" iyz="0.0" izz="0.001"/>
+			</inertial>
 		<visual>
 		    <origin xyz="0 0.005 0.0065" rpy="0 0 1.57" />
@@ -106,15 +110,16 @@
 		</visual>
 		<collision>
-		  <geometry>
-		    <mesh filename="package://mlp3240_description/mesh/visual/front_w_box.stl" scale="0.001 0.001 0.001"/>
-		  </geometry>
-	        </collision>
+			<origin xyz="0 0.005 0.0065" rpy="0 0 1.57" />
+		  	<geometry>
+		    	<mesh filename="package://mlp3240_description/mesh/visual/front_w_box.stl" scale="0.001 0.001 0.001"/>
+		  	</geometry>
+	    </collision>
 	    </link>
 	    <link name="${prefix}top">
 	    	<inertial>
-			<origin xyz="0 0 0" rpy="0 0 0"/>
-			<mass value="0.001"/>
-			<inertia ixx="0.01" ixy="0.0" ixz="0.0" iyy="0.001" iyz="0.0" izz="0.001"/>
-		 </inertial>
+				<origin xyz="0 0 0" rpy="0 0 0"/>
+				<mass value="0.001"/>
+				<inertia ixx="0.01" ixy="0.0" ixz="0.0" iyy="0.001" iyz="0.0" izz="0.001"/>
+			</inertial>
 		<visual>
 		    <origin xyz="0 0 0.006" rpy="0 0 1.57" />
@@ -127,15 +132,16 @@
 		</visual>
 		<collision>
-		  <geometry>
-		    <mesh filename="package://mlp3240_description/mesh/visual/top.stl" scale="0.001 0.001 0.001"/>
-		  </geometry>
-	        </collision>
+			<origin xyz="0 0 0.006" rpy="0 0 1.57" />
+		  	<geometry>
+		    	<mesh filename="package://mlp3240_description/mesh/visual/top.stl" scale="0.001 0.001 0.001"/>
+		  	</geometry>
+	    </collision>
 	    </link>
 	    <link name="${prefix}finger1">
 	    	<inertial>
-			<origin xyz="0 0 0" rpy="0 0 0"/>
-			<mass value="0.001"/>
-			<inertia ixx="0.001" ixy="0.0" ixz="0.0" iyy="0.001" iyz="0.0" izz="0.001"/>
-		 </inertial>
+				<origin xyz="0 0 0" rpy="0 0 0"/>
+				<mass value="0.001"/>
+				<inertia ixx="0.001" ixy="0.0" ixz="0.0" iyy="0.001" iyz="0.0" izz="0.001"/>
+			</inertial>
 		<visual>
 		    <origin xyz="0.015 0 0.001" rpy="0 0 1.57" />
@@ -146,15 +152,16 @@
 		</visual>
 		<collision>
-		  <geometry>
-		    <mesh filename="package://mlp3240_description/mesh/visual/finger_1.stl" scale="0.001 0.001 0.001"/>
-		  </geometry>
-	        </collision>
+			<origin xyz="0.015 0 0.001" rpy="0 0 1.57" />
+		  	<geometry>
+		    	<mesh filename="package://mlp3240_description/mesh/visual/finger_1.stl" scale="0.001 0.001 0.001"/>
+		  	</geometry>
+	    </collision>
 	    </link>
 	    <link name="${prefix}finger2">
 	    	<inertial>
-			<origin xyz="0 0 0" rpy="0 0 0"/>
-			<mass value="0.001"/>
-			<inertia ixx="0.001" ixy="0.0" ixz="0.0" iyy="0.001" iyz="0.0" izz="0.001"/>
-		 </inertial>
+				<origin xyz="0 0 0" rpy="0 0 0"/>
+				<mass value="0.001"/>
+				<inertia ixx="0.001" ixy="0.0" ixz="0.0" iyy="0.001" iyz="0.0" izz="0.001"/>
+			</inertial>
 		<visual>
 		    <origin xyz="0.015 0 0.001" rpy="0 0 1.57" />
@@ -165,8 +172,9 @@
 		</visual>
 		<collision>
-		  <geometry>
-		    <mesh filename="package://mlp3240_description/mesh/visual/finger_2.stl" scale="0.001 0.001 0.001"/>
-		  </geometry>
-	        </collision>
+			<origin xyz="0.015 0 0.001" rpy="0 0 1.57" />
+		  	<geometry>
+		    	<mesh filename="package://mlp3240_description/mesh/visual/finger_2.stl" scale="0.001 0.001 0.001"/>
+		  	</geometry>
+	    </collision>
 	    </link>
 	<joint name="${prefix}base_to_left_joint" type="fixed">
@@ -227,4 +235,21 @@
 		</plugin>
 	</gazebo>
+	<!-- Improve grasping physics -->
+    <gazebo reference="${prefix}finger1">
+      <kp>1000000.0</kp>
+      <kd>0.0</kd>
+      <mu1>1.0</mu1>
+      <mu2>1.0</mu2>
+      <minDepth>0.001</minDepth>
+	  <maxVel>1000</maxVel>
+    </gazebo>
+    <gazebo reference="${prefix}finger2">
+      <kp>500000.0</kp>
+      <kd>0.0</kd>
+      <mu1>1.0</mu1>
+      <mu2>1.0</mu2>
+      <minDepth>0.001</minDepth>
+	  <maxVel>1000</maxVel>
+    </gazebo>
 	</xacro:macro>
 </robot>

Commit message: Friction Improvement

File: src/src/mlp3240/mlp3240_description/urdf/mlp3240_macro.xacro (robot description, xacro)
@@ -140,7 +140,7 @@
 	    <link name="${prefix}finger1">
 	    	<inertial>
-				<origin xyz="0 0 0" rpy="0 0 0"/>
-				<mass value="0.001"/>
-				<inertia ixx="0.001" ixy="0.0" ixz="0.0" iyy="0.001" iyz="0.0" izz="0.001"/>
+				<origin xyz="0.015 0 0.02" rpy="0 0 1.57" />
+				<mass value="0.01"/>
+				<inertia ixx="0.0000006" ixy="0.0" ixz="0.0" iyy="0.000001" iyz="0.0" izz="0.0000005"/>
 			</inertial>
 		<visual>
@@ -156,11 +156,19 @@
 		    	<mesh filename="package://mlp3240_description/mesh/visual/finger_1.stl" scale="0.001 0.001 0.001"/>
 		  	</geometry>
+			<surface>
+				<friction>
+					<ode>
+						<mu>1000</mu>
+						<mu2>1000</mu2>
+					</ode>
+				</friction>
+          	</surface>
 	    </collision>
 	    </link>
 	    <link name="${prefix}finger2">
 	    	<inertial>
-				<origin xyz="0 0 0" rpy="0 0 0"/>
-				<mass value="0.001"/>
-				<inertia ixx="0.001" ixy="0.0" ixz="0.0" iyy="0.001" iyz="0.0" izz="0.001"/>
+				<origin xyz="0.015 0 0.02" rpy="0 0 1.57" />
+				<mass value="0.01"/>
+				<inertia ixx="0.0000006" ixy="0.0" ixz="0.0" iyy="0.000001" iyz="0.0" izz="0.0000005"/>
 			</inertial>
 		<visual>
@@ -176,4 +184,12 @@
 		    	<mesh filename="package://mlp3240_description/mesh/visual/finger_2.stl" scale="0.001 0.001 0.001"/>
 		  	</geometry>
+			<surface>
+				<friction>
+					<ode>
+						<mu>1000</mu>
+						<mu2>1000</mu2>
+					</ode>
+				</friction>
+          	</surface>
 	    </collision>
 	    </link>
@@ -237,8 +253,8 @@
 	<!-- Improve grasping physics -->
     <gazebo reference="${prefix}finger1">
-      <kp>1000000.0</kp>
+      <kp>500000.0</kp>
       <kd>0.0</kd>
-      <mu1>1.0</mu1>
-      <mu2>1.0</mu2>
+      <mu1>10000</mu1>
+      <mu2>10000</mu2>
       <minDepth>0.001</minDepth>
 	  <maxVel>1000</maxVel>
@@ -247,6 +263,6 @@
       <kp>500000.0</kp>
       <kd>0.0</kd>
-      <mu1>1.0</mu1>
-      <mu2>1.0</mu2>
+      <mu1>10000</mu1>
+      <mu2>10000</mu2>
       <minDepth>0.001</minDepth>
 	  <maxVel>1000</maxVel>

File: src/src/ur5e_mlp3240_task/urdf/ur5e_mlp3240.urdf.xacro (robot description, xacro)
@@ -24,5 +24,5 @@
 	<link name="ee_tool"/>
 	<joint name="ee_link_to_ee_tool" type="fixed">
-	      <origin xyz="0.01 0 0" rpy="0 0 0"/>
+	      <origin xyz="0.007 0 0" rpy="0 0 0"/>
 	      <parent link="ee_link"/>
 	      <child link="ee_tool"/>
@@ -34,8 +34,8 @@
   	<plugin name="gazebo_grasp_fix" filename="libgazebo_grasp_fix.so">
 	  	<arm>
-	  		<arm_name>mlp3240_gripper</arm_name>
+	  		<arm_name>robot</arm_name>
 	  		<palm_link>wrist_3_link</palm_link>
-	      		<gripper_link>finger1</gripper_link>
-	      		<gripper_link>finger2</gripper_link>
+	      	<gripper_link>finger1</gripper_link>
+	      	<gripper_link>finger2</gripper_link>
 	  	</arm>
   	<forces_angle_tolerance>100</forces_angle_tolerance>
@@ -43,5 +43,5 @@
   	<grip_count_threshold>1</grip_count_threshold>
   	<max_grip_count>5</max_grip_count>
-  	<release_tolerance>0.01</release_tolerance>
+  	<release_tolerance>0.005</release_tolerance>
   	<disable_collisions_on_attach>true</disable_collisions_on_attach>
   	<contact_topic>__default_topic__</contact_topic>

Commit message: better grasp

File: src/src/mlp3240/mlp3240_description/urdf/mlp3240_macro.xacro (robot description, xacro)
@@ -2,8 +2,8 @@
 <robot  xmlns:xacro="http://ros.org/wiki/xacro">
 	<xacro:macro name="mlp3240" params="prefix ">
-	<xacro:property name="physical_parameters" value="${load_yaml('$(find mlp3240_description)/config/physical_params.yaml')}"/>
-	<material name="white">
-	    <color rgba="1 1 1 1"/>
-	</material>
+		<xacro:property name="physical_parameters" value="${load_yaml('$(find mlp3240_description)/config/physical_params.yaml')}"/>
+		<material name="white">
+			<color rgba="1 1 1 1"/>
+		</material>
 	    <link name="${prefix}base_link_gripper">
 		<inertial>
@@ -140,7 +140,7 @@
 	    <link name="${prefix}finger1">
 	    	<inertial>
-				<origin xyz="0.015 0 0.02" rpy="0 0 1.57" />
+				<origin xyz="0.015 0 0.015" rpy="0 0 1.57" />
 				<mass value="0.01"/>
-				<inertia ixx="0.0000006" ixy="0.0" ixz="0.0" iyy="0.000001" iyz="0.0" izz="0.0000005"/>
+				<inertia ixx="0.0000015" ixy="0.0" ixz="0.0" iyy="0.0000015" iyz="0.0" izz="0.0000005"/>
 			</inertial>
 		<visual>
@@ -156,116 +156,152 @@
 		    	<mesh filename="package://mlp3240_description/mesh/visual/finger_1.stl" scale="0.001 0.001 0.001"/>
 		  	</geometry>
+	    </collision>
+	    </link>
+	    <link name="${prefix}finger2">
+	    	<inertial>
+				<origin xyz="0.015 0 0.01" rpy="0 0 1.57" />
+				<mass value="0.01"/>
+				<inertia ixx="0.0000015" ixy="0.0" ixz="0.0" iyy="0.0000015" iyz="0.0" izz="0.0000005"/>
+			</inertial>
+		<visual>
+		    <origin xyz="0.015 0 0.0015" rpy="0 0 1.57" />
+		    <geometry>
+		        <mesh filename="package://mlp3240_description/mesh/visual/finger_2.stl" scale="0.001 0.001 0.001"/>
+		    </geometry>
+		    <material name="white"/>
+		</visual>
+		<collision>
+			<origin xyz="0.015 0 0.001" rpy="0 0 1.57" />
+		  	<geometry>
+		    	<mesh filename="package://mlp3240_description/mesh/visual/finger_2.stl" scale="0.001 0.001 0.001"/>
+		  	</geometry>
+			<!--
 			<surface>
 				<friction>
 					<ode>
-						<mu>1000</mu>
-						<mu2>1000</mu2>
+						<mu>100.0</mu>
+						<mu2>100.0</mu2>
 					</ode>
 				</friction>
+				<contact>
+					<ode>
+						<kp>1000000.0</kp>
+						<kd>100.0</kd>
+						<max_vel>1.0</max_vel>
+						<min_depth>0.002</min_depth>
+					</ode>
+              	</contact>
           	</surface>
-	    </collision>
-	    </link>
-	    <link name="${prefix}finger2">
-	    	<inertial>
-				<origin xyz="0.015 0 0.02" rpy="0 0 1.57" />
-				<mass value="0.01"/>
-				<inertia ixx="0.0000006" ixy="0.0" ixz="0.0" iyy="0.000001" iyz="0.0" izz="0.0000005"/>
-			</inertial>
-		<visual>
-		    <origin xyz="0.015 0 0.001" rpy="0 0 1.57" />
-		    <geometry>
-		        <mesh filename="package://mlp3240_description/mesh/visual/finger_2.stl" scale="0.001 0.001 0.001"/>
-		    </geometry>
-		    <material name="white"/>
-		</visual>
-		<collision>
-			<origin xyz="0.015 0 0.001" rpy="0 0 1.57" />
-		  	<geometry>
-		    	<mesh filename="package://mlp3240_description/mesh/visual/finger_2.stl" scale="0.001 0.001 0.001"/>
-		  	</geometry>
-			<surface>
-				<friction>
-					<ode>
-						<mu>1000</mu>
-						<mu2>1000</mu2>
-					</ode>
-				</friction>
-          	</surface>
-	    </collision>
-	    </link>
-	<joint name="${prefix}base_to_left_joint" type="fixed">
-	    <parent link="${prefix}base_link_gripper"/>
-	    <child link="${prefix}left"/>
-	    <origin xyz="${physical_parameters['base_x']/2} 0 0.015" rpy='0 0 0'/>
-	</joint>
-	<joint name="${prefix}base_to_right_joint" type="fixed">
-	    <parent link="${prefix}base_link_gripper"/>
-	    <child link="${prefix}right"/>
-	    <origin xyz="-${physical_parameters['base_x']/2} 0 0.015" rpy='0 0 0'/>
-	</joint>
-	<joint name="${prefix}base_to_front_joint" type="fixed">
-	    <parent link="${prefix}base_link_gripper"/>
-	    <child link="${prefix}front"/>
-	    <origin xyz="0 ${physical_parameters['base_y']/2} 0.015" rpy='0 0 0'/>
-	</joint>
-	<joint name="${prefix}base_to_back_joint" type="fixed">
-	    <parent link="${prefix}base_link_gripper"/>
-	    <child link="${prefix}back"/>
-	    <origin xyz="0 -${physical_parameters['base_y']/2} 0.015" rpy='0 0 0'/>
-	</joint>
-	<joint name="${prefix}left_to_top_joint" type="fixed">
-	    <parent link="${prefix}left"/>
-	    <child link="${prefix}top"/>
-	    <origin xyz="-${physical_parameters['left_y']} 0 0.03" rpy='0 0 0'/>
-	</joint>
-	<joint name="${prefix}top_to_finger1_joint" type="prismatic">
-	    <parent link="${prefix}top"/>
-	    <child link="${prefix}finger1"/>
-	    <origin xyz="${physical_parameters['top_x']/2 - 0.005} 0 0.0211" rpy='0 0 -3.14'/>
-	    <limit upper="0.0336" lower="0.0" effort="300" velocity="1"/>
-	</joint>
-	<joint name="${prefix}top_to_finger2_joint" type="prismatic">
-	    <parent link="${prefix}top"/>
-	    <child link="${prefix}finger2"/>
-	    <origin xyz="-${physical_parameters['top_x']/2 - 0.005} 0 0.021" rpy='0 0 0'/>
-	    <limit upper="0.0336" lower="0.0" effort="300" velocity="1"/>
-	    <mimic joint="${prefix}top_to_finger1_joint" multiplier="1.0" offset="0.0" />
-	</joint>
-	<!-- <xacro:macro name="mlp3240_gripper_transmission" params="${prefix}"/> -->
-	<!-- Transmission for ROS control -->
-	<transmission name="${prefix}top_to_finger1_joint_trans">
-	      <type>transmission_interface/SimpleTransmission</type>
-	      <joint name="${prefix}top_to_finger1_joint">
-			<hardwareInterface>hardware_interface/EffortJointInterface</hardwareInterface>
-	      </joint>
-	      <actuator name="${prefix}top_to_finger1_joint_motor">
-			<mechanicalReduction>1</mechanicalReduction>
-			<hardwareInterface>hardware_interface/EfforJointInterface</hardwareInterface>
-	      </actuator>
-	</transmission>
-	<!-- Mimic joints -->
-	<gazebo>
-		<plugin filename="libgazebo_mimic_joint_plugin.so" name="${prefix}mimic_top_to_finger1_joint">
-			<joint>${prefix}top_to_finger1_joint</joint>
-			<mimicJoint>${prefix}top_to_finger2_joint</mimicJoint>
-		</plugin>
-	</gazebo>
-	<!-- Improve grasping physics -->
-    <gazebo reference="${prefix}finger1">
-      <kp>500000.0</kp>
-      <kd>0.0</kd>
-      <mu1>10000</mu1>
-      <mu2>10000</mu2>
-      <minDepth>0.001</minDepth>
-	  <maxVel>1000</maxVel>
-    </gazebo>
-    <gazebo reference="${prefix}finger2">
-      <kp>500000.0</kp>
-      <kd>0.0</kd>
-      <mu1>10000</mu1>
-      <mu2>10000</mu2>
-      <minDepth>0.001</minDepth>
-	  <maxVel>1000</maxVel>
-    </gazebo>
+			-->
+	    </collision>
+	    </link>
+		<joint name="${prefix}base_to_left_joint" type="fixed">
+			<parent link="${prefix}base_link_gripper"/>
+			<child link="${prefix}left"/>
+			<origin xyz="${physical_parameters['base_x']/2} 0 0.015" rpy='0 0 0'/>
+		</joint>
+		<joint name="${prefix}base_to_right_joint" type="fixed">
+			<parent link="${prefix}base_link_gripper"/>
+			<child link="${prefix}right"/>
+			<origin xyz="-${physical_parameters['base_x']/2} 0 0.015" rpy='0 0 0'/>
+		</joint>
+		<joint name="${prefix}base_to_front_joint" type="fixed">
+			<parent link="${prefix}base_link_gripper"/>
+			<child link="${prefix}front"/>
+			<origin xyz="0 ${physical_parameters['base_y']/2} 0.015" rpy='0 0 0'/>
+		</joint>
+		<joint name="${prefix}base_to_back_joint" type="fixed">
+			<parent link="${prefix}base_link_gripper"/>
+			<child link="${prefix}back"/>
+			<origin xyz="0 -${physical_parameters['base_y']/2} 0.015" rpy='0 0 0'/>
+		</joint>
+		<joint name="${prefix}left_to_top_joint" type="fixed">
+			<parent link="${prefix}left"/>
+			<child link="${prefix}top"/>
+			<origin xyz="-${physical_parameters['left_y']} 0 0.03" rpy='0 0 0'/>
+		</joint>
+		<joint name="${prefix}top_to_finger1_joint" type="prismatic">
+			<parent link="${prefix}top"/>
+			<child link="${prefix}finger1"/>
+			<origin xyz="${physical_parameters['top_x']/2 - 0.005} 0 0.0211" rpy='0 0 -3.14'/>
+			<limit upper="0.0336" lower="0.0" effort="300" velocity="1"/>
+		</joint>
+		<joint name="${prefix}top_to_finger2_joint" type="prismatic">
+			<parent link="${prefix}top"/>
+			<child link="${prefix}finger2"/>
+			<origin xyz="-${physical_parameters['top_x']/2 - 0.005} 0 0.021" rpy='0 0 0'/>
+			<limit upper="0.0336" lower="0.0" effort="300" velocity="1"/>
+			<mimic joint="${prefix}top_to_finger1_joint" multiplier="1.0" offset="0.0" />
+		</joint>
+		<!-- Transmission for ROS control -->
+		<transmission name="${prefix}top_to_finger1_joint_trans">
+			<type>transmission_interface/SimpleTransmission</type>
+			<joint name="${prefix}top_to_finger1_joint">
+				<hardwareInterface>hardware_interface/EffortJointInterface</hardwareInterface>
+			</joint>
+			<actuator name="${prefix}top_to_finger1_joint_motor">
+				<mechanicalReduction>1</mechanicalReduction>
+				<hardwareInterface>hardware_interface/EfforJointInterface</hardwareInterface>
+			</actuator>
+		</transmission>
+		<!-- Mimic joints -->
+		<gazebo>
+			<plugin filename="libgazebo_mimic_joint_plugin.so" name="${prefix}mimic_top_to_finger1_joint">
+				<joint>${prefix}top_to_finger1_joint</joint>
+				<mimicJoint>${prefix}top_to_finger2_joint</mimicJoint>
+			</plugin>
+		</gazebo>
+		<!-- Improve grasping physics -->
+		<gazebo reference="${prefix}finger1">
+			<kp>1000000.0</kp>
+			<kd>10.0</kd>
+			<mu1>100.0</mu1>
+			<mu2>100.0</mu2>
+			<minDepth>0.001</minDepth>
+			<maxVel>1000</maxVel>
+		</gazebo>
+		<gazebo reference="${prefix}finger2">
+			<kp>500000.0</kp>
+			<kd>10.0</kd>
+			<mu1>100.0</mu1>
+			<mu2>100.0</mu2>
+			<minDepth>0.001</minDepth>
+			<maxVel>1000</maxVel>
+		</gazebo>
+		<gazebo>
+	  		<plugin name="gazebo_ros_control" filename="libgazebo_ros_control.so" />
+    	</gazebo>
+		<!-- to get grasping properly works on Gazebo -->
+		<gazebo>
+			<plugin name="gazebo_grasp_fix" filename="libgazebo_grasp_fix.so">
+				<arm>
+					<arm_name>robot_arm</arm_name>
+					<palm_link>wrist_3_link</palm_link>
+					<gripper_link>finger1</gripper_link>
+					<gripper_link>finger2</gripper_link>
+				</arm>
+				<forces_angle_tolerance>90</forces_angle_tolerance>
+				<update_rate>4</update_rate>
+				<grip_count_threshold>1</grip_count_threshold>
+				<max_grip_count>8</max_grip_count>
+				<release_tolerance>0.005</release_tolerance>
+				<disable_collisions_on_attach>false</disable_collisions_on_attach>
+				<contact_topic>__default_topic__</contact_topic>
+			</plugin>
+		</gazebo>
+		<!--
+		<gazebo>
+			<gripper name="grasping">
+				<grasp_check>
+					<attach_steps>1</attach_steps>
+					<detach_steps>10</detach_steps>
+					<min_contact_count>1</min_contact_count>
+				</grasp_check>
+				<palm_link>wrist_3_link</palm_link>
+				<gripper_link>finger1</gripper_link>
+				<gripper_link>finger2</gripper_link>
+			</gripper>
+		</gazebo>
+		-->
 	</xacro:macro>
 </robot>

File: src/src/ur5e_mlp3240_task/urdf/ur5e_mlp3240.urdf.xacro (robot description, xacro)
@@ -24,5 +24,5 @@
 	<link name="ee_tool"/>
 	<joint name="ee_link_to_ee_tool" type="fixed">
-	      <origin xyz="0.007 0 0" rpy="0 0 0"/>
+	      <origin xyz="0.01 0 0" rpy="0 0 0"/>
 	      <parent link="ee_link"/>
 	      <child link="ee_tool"/>
@@ -30,24 +30,3 @@
 </xacro:macro>
 <xacro:ur5e_mlp3240 prefix=""/>
-	<!-- to properly work on Gazebo -->
-    <gazebo>
-  	<plugin name="gazebo_grasp_fix" filename="libgazebo_grasp_fix.so">
-	  	<arm>
-	  		<arm_name>robot</arm_name>
-	  		<palm_link>wrist_3_link</palm_link>
-	      	<gripper_link>finger1</gripper_link>
-	      	<gripper_link>finger2</gripper_link>
-	  	</arm>
-  	<forces_angle_tolerance>100</forces_angle_tolerance>
-  	<update_rate>10</update_rate>
-  	<grip_count_threshold>1</grip_count_threshold>
-  	<max_grip_count>5</max_grip_count>
-  	<release_tolerance>0.005</release_tolerance>
-  	<disable_collisions_on_attach>true</disable_collisions_on_attach>
-  	<contact_topic>__default_topic__</contact_topic>
-  	</plugin>
-    </gazebo>
-    <gazebo>
-	  <plugin name="gazebo_ros_control" filename="libgazebo_ros_control.so" />
-    </gazebo>
 </robot>
