Commit message: Almost Working Task

File: src/src/mlp3240/mlp3240_description/urdf/mlp3240_macro.xacro (robot description, xacro)
@@ -108,11 +108,11 @@
 		        <color rgba="${61/255} ${61/255} ${61/255} 1.0"/>
 		    </material>
-		</visual>
-		<collision>
-			<origin xyz="0 0.005 0.0065" rpy="0 0 1.57" />
-		  	<geometry>
-		    	<mesh filename="package://mlp3240_description/mesh/visual/front_w_box.stl" scale="0.001 0.001 0.001"/>
-		  	</geometry>
-	    </collision>
+			</visual>
+			<collision>
+				<origin xyz="0 0.005 0.0065" rpy="0 0 1.57" />
+				<geometry>
+					<mesh filename="package://mlp3240_description/mesh/visual/front_w_box.stl" scale="0.001 0.001 0.001"/>
+				</geometry>
+			</collision>
 	    </link>
 	    <link name="${prefix}top">
@@ -122,77 +122,73 @@
 				<inertia ixx="0.01" ixy="0.0" ixz="0.0" iyy="0.001" iyz="0.0" izz="0.001"/>
 			</inertial>
-		<visual>
-		    <origin xyz="0 0 0.006" rpy="0 0 1.57" />
-		    <geometry>
-		        <mesh filename="package://mlp3240_description/mesh/visual/top.stl" scale="0.001 0.001 0.001"/>
-		    </geometry>
-		    <material name="black">
-		        <color rgba="${61/255} ${61/255} ${61/255} 1.0"/>
-		    </material>
-		</visual>
-		<collision>
-			<origin xyz="0 0 0.006" rpy="0 0 1.57" />
-		  	<geometry>
-		    	<mesh filename="package://mlp3240_description/mesh/visual/top.stl" scale="0.001 0.001 0.001"/>
-		  	</geometry>
-	    </collision>
+			<visual>
+				<origin xyz="0 0 0.006" rpy="0 0 1.57" />
+				<geometry>
+					<mesh filename="package://mlp3240_description/mesh/visual/top.stl" scale="0.001 0.001 0.001"/>
+				</geometry>
+				<material name="black">
+					<color rgba="${61/255} ${61/255} ${61/255} 1.0"/>
+				</material>
+			</visual>
+			<collision>
+				<origin xyz="0 0 0.006" rpy="0 0 1.57" />
+				<geometry>
+					<mesh filename="package://mlp3240_description/mesh/visual/top.stl" scale="0.001 0.001 0.001"/>
+				</geometry>
+			</collision>
 	    </link>
 	    <link name="${prefix}finger1">
 	    	<inertial>
-				<origin xyz="0.015 0 0.015" rpy="0 0 1.57" />
-				<mass value="0.01"/>
-				<inertia ixx="0.0000015" ixy="0.0" ixz="0.0" iyy="0.0000015" iyz="0.0" izz="0.0000005"/>
-			</inertial>
-		<visual>
-		    <origin xyz="0.015 0 0.001" rpy="0 0 1.57" />
-		    <geometry>
-		        <mesh filename="package://mlp3240_description/mesh/visual/finger_1.stl" scale="0.001 0.001 0.001"/>
-		    </geometry>
-		    <material name="white"/>
-		</visual>
-		<collision>
-			<origin xyz="0.015 0 0.001" rpy="0 0 1.57" />
-		  	<geometry>
-		    	<mesh filename="package://mlp3240_description/mesh/visual/finger_1.stl" scale="0.001 0.001 0.001"/>
-		  	</geometry>
-	    </collision>
+				<origin xyz="0.015 0 0.015" rpy="0 0 0" />
+				<mass value="0.1"/>
+				<inertia ixx="0.000015417" ixy="0.0" ixz="0.0" iyy="0.000010232" iyz="0.0" izz="0.000005232"/>
+			</inertial>
+			<visual>
+				<origin xyz="0.015 0 0.001" rpy="0 0 1.57" />
+				<geometry>
+					<mesh filename="package://mlp3240_description/mesh/visual/finger_1.stl" scale="0.001 0.001 0.001"/>
+				</geometry>
+				<material name="white"/>
+			</visual>
+			<collision>
+				<origin xyz="0.015 0 0.015" rpy="0 0 0" />
+				<geometry>
+        			<box size="0.0017 0.025 0.035" />
+		  		</geometry>
+			</collision>
+			<!-- bad mesh causes bad physics while collision
+			<collision>
+				<origin xyz="0.015 0 0.001" rpy="0 0 1.57" />
+				<geometry>
+					<mesh filename="package://mlp3240_description/mesh/visual/finger_1.stl" scale="0.001 0.001 0.001"/>
+				</geometry>
+			</collision>
+			-->
 	    </link>
 	    <link name="${prefix}finger2">
 	    	<inertial>
-				<origin xyz="0.015 0 0.01" rpy="0 0 1.57" />
-				<mass value="0.01"/>
-				<inertia ixx="0.0000015" ixy="0.0" ixz="0.0" iyy="0.0000015" iyz="0.0" izz="0.0000005"/>
-			</inertial>
-		<visual>
-		    <origin xyz="0.015 0 0.0015" rpy="0 0 1.57" />
-		    <geometry>
-		        <mesh filename="package://mlp3240_description/mesh/visual/finger_2.stl" scale="0.001 0.001 0.001"/>
-		    </geometry>
-		    <material name="white"/>
-		</visual>
-		<collision>
-			<origin xyz="0.015 0 0.001" rpy="0 0 1.57" />
-		  	<geometry>
-		    	<mesh filename="package://mlp3240_description/mesh/visual/finger_2.stl" scale="0.001 0.001 0.001"/>
-		  	</geometry>
-			<!--
-			<surface>
-				<friction>
-					<ode>
-						<mu>100.0</mu>
-						<mu2>100.0</mu2>
-					</ode>
-				</friction>
-				<contact>
-					<ode>
-						<kp>1000000.0</kp>
-						<kd>100.0</kd>
-						<max_vel>1.0</max_vel>
-						<min_depth>0.002</min_depth>
-					</ode>
-              	</contact>
-          	</surface>
-			-->
-	    </collision>
+				<origin xyz="0.015 0 0.015" rpy="0 0 0" />
+				<mass value="0.1"/>
+				<inertia ixx="0.000015417" ixy="0.0" ixz="0.0" iyy="0.000010232" iyz="0.0" izz="0.000005232"/>
+			</inertial>
+			<visual>
+				<origin xyz="0.015 0 0.0015" rpy="0 0 1.57" />
+				<geometry>
+					<mesh filename="package://mlp3240_description/mesh/visual/finger_2.stl" scale="0.001 0.001 0.001"/>
+				</geometry>
+				<material name="white"/>
+			</visual>
+			<collision>
+				<origin xyz="0.015 0 0.015" rpy="0 0 0" />
+				<geometry>
+        			<box size="0.0017 0.025 0.035" />
+		  		</geometry>
+				<!-- bad mesh causes bad physics while collision
+				<origin xyz="0.015 0 0.001" rpy="0 0 1.57" />
+				<geometry>
+		    		<mesh filename="package://mlp3240_description/mesh/visual/finger_2.stl" scale="0.001 0.001 0.001"/>
+		  		</geometry>
+				-->
+	    	</collision>
 	    </link>
 		<joint name="${prefix}base_to_left_joint" type="fixed">
@@ -254,4 +250,19 @@
 		<!-- Improve grasping physics -->
 		<gazebo reference="${prefix}finger1">
+			<collision name="finger1_collision">
+			<surface>
+				<friction>
+					<torsional>
+						<coefficient>10.0</coefficient>
+						<use_patch_radius>true</use_patch_radius>
+						<patch_radius>0.05</patch_radius>
+					</torsional>
+				</friction>
+				<contact>
+					<poissons_ratio>0.5</poissons_ratio>
+					<elastic_modulus>1e8</elastic_modulus>
+				</contact>
+			</surface>
+			</collision>
 			<kp>1000000.0</kp>
 			<kd>10.0</kd>
@@ -262,5 +273,20 @@
 		</gazebo>
 		<gazebo reference="${prefix}finger2">
-			<kp>500000.0</kp>
+			<collision name="finger2_collision">
+			<surface>
+				<friction>
+					<torsional>
+						<coefficient>10.0</coefficient>
+						<use_patch_radius>true</use_patch_radius>
+						<patch_radius>0.05</patch_radius>
+					</torsional>
+				</friction>
+				<contact>
+					<poissons_ratio>0.5</poissons_ratio>
+					<elastic_modulus>1e8</elastic_modulus>
+				</contact>
+			</surface>
+			</collision>
+			<kp>1000000.0</kp>
 			<kd>10.0</kd>
 			<mu1>100.0</mu1>
@@ -281,10 +307,10 @@
 					<gripper_link>finger2</gripper_link>
 				</arm>
-				<forces_angle_tolerance>90</forces_angle_tolerance>
-				<update_rate>4</update_rate>
+				<forces_angle_tolerance>100</forces_angle_tolerance>
+				<update_rate>10</update_rate>
 				<grip_count_threshold>1</grip_count_threshold>
-				<max_grip_count>8</max_grip_count>
-				<release_tolerance>0.005</release_tolerance>
-				<disable_collisions_on_attach>false</disable_collisions_on_attach>
+				<max_grip_count>10</max_grip_count>
+				<release_tolerance>0.001</release_tolerance>
+				<disable_collisions_on_attach>true</disable_collisions_on_attach>
 				<contact_topic>__default_topic__</contact_topic>
 			</plugin>

File: src/src/ur5e_mlp3240_task/urdf/ur5e_mlp3240.urdf.xacro (robot description, xacro)
@@ -24,5 +24,5 @@
 	<link name="ee_tool"/>
 	<joint name="ee_link_to_ee_tool" type="fixed">
-	      <origin xyz="0.01 0 0" rpy="0 0 0"/>
+	      <origin xyz="0.105 0 0" rpy="0 0 0"/>
 	      <parent link="ee_link"/>
 	      <child link="ee_tool"/>
